File: board/board.kicad_pcb (KiCad board)
At the start: 2 copper layers, 21 x 13 mm, 1 part

Commit message: initial
Parts:
- added C2: 10uF, Capacitor_SMD:C_0603_1608Metric, F.Cu at (149.7, 101.5)
- added C3: 10uF, Capacitor_SMD:C_0603_1608Metric, F.Cu at (149.7, 100.0)
- added C4: 100nF, Capacitor_SMD:C_0402_1005Metric, F.Cu at (149.2, 98.7)
- added C5: 22uF, Capacitor_SMD:C_0603_1608Metric, F.Cu at (148.6, 92.8)
- added C58: 100nF, Capacitor_SMD:C_0402_1005Metric, F.Cu at (149.1, 95.7)
- added C6: 22uF, Capacitor_SMD:C_0603_1608Metric, F.Cu at (148.6, 94.3)
- added J1: 000_3.3v_5v, on_edge:on_edge_2x05_device, F.Cu at (140.0, 96.5)
- added J2: 000_3.3v_5v, on_edge:on_edge_2x05_host, F.Cu at (161.0, 96.5)
- added L1: MWSA0503S-3R3MT, Inductor_SMD:L_Sunlord_MWSA0503S, F.Cu at (153.1, 95.9)
- added R1: 47k, Resistor_SMD:R_0402_1005Metric, F.Cu at (146.1, 97.1)
- added R12: 10k, Resistor_SMD:R_0402_1005Metric, F.Cu at (146.1, 95.1)
- added R13: 49.9k, Resistor_SMD:R_0402_1005Metric, F.Cu at (146.1, 98.1)
- added R14: 510k, Resistor_SMD:R_0402_1005Metric, F.Cu at (146.1, 99.1)
- added R2: 12k, Resistor_SMD:R_0402_1005Metric, F.Cu at (146.1, 96.1)
- added R57: 10k, Resistor_SMD:R_0402_1005Metric, F.Cu at (146.1, 100.1)
- added U7: TPS564257DRLR, Package_TO_SOT_SMD:SOT-563, F.Cu at (148.9, 97.2)
- LOGO1: moved to B.Cu
- moved LOGO1 2.60 mm to (150.0, 96.4), turned to 180 degrees
Routing:
- net GND: track 0.00 -> 55.4 mm, vias 0 -> 26
- net /buck/3.3V: track 0.00 -> 27.4 mm, vias 0 -> 1
- net /buck/Vin: track 0.00 -> 14.5 mm, vias 0 -> 2
- net Net-(U7-FB): track 0.00 -> 4.15 mm
- net /buck/sw: track 0.00 -> 3.27 mm
- net /buck/EN: track 0.00 -> 2.60 mm
- net /buck/PG: track 0.00 -> 2.24 mm
- added copper zone on B.Cu, net GND
- added copper zone on F.Cu, net GND
Other:
- outline, holes or cut-outs redrawn
- board text added: "osf.000"
- board text added: "osf.b169.v1.0"
