File: board/board.kicad_sch (KiCad schematic)
At the start: 1 part

Commit message: initial
Parts:
- added J1: 000_3.3v_5v, on_edge:on_edge_2x05_device, symbol put_on_edge:000_3.3v_5v
- added J2: 000_3.3v_5v, on_edge:on_edge_2x05_host, symbol put_on_edge:000_3.3v_5v
- added R1: 47k, Resistor_SMD:R_0402_1005Metric, symbol Device:R_Small
- added R2: 12k, Resistor_SMD:R_0402_1005Metric, symbol Device:R_Small
Connections:
- net GND: now also J1.1 (GND), J2.1 (GND), R2.1
- new net buck/3.3V: J2.9 (3.3V)
- new net buck/EN: R1.1, R2.2
- new net buck/Vin: J1.10 (5V), R1.2
Other:
- sheet implementation renamed buck
- sheet buck: file implementation.kicad_sch -> buck.kicad_sch
- sheet buck ports: added 3.3V, EN, Vin; removed none
- note removed: "Input connectors go here"
- note removed: "Output connectors go here"
